Commit message: nit path

File: simulation/follower.urdf (robot description, URDF)
Before this commit: robot follower, 7 links, 6 joints
Links:
- link base_link: geometry collision mesh filename=./meshes/base_link.STL; visual mesh filename=./meshes/base_link.STL
- link link_1: geometry collision mesh filename=./meshes/link_1.STL; visual mesh filename=./meshes/link_1.STL
- link link_2: geometry collision mesh filename=./meshes/link_2.STL; visual mesh filename=./meshes/link_2.STL
- link link_3: geometry collision mesh filename=./meshes/link_3.STL; visual mesh filename=./meshes/link_3.STL
- link link_4: geometry collision mesh filename=./meshes/link_4.STL; visual mesh filename=./meshes/link_4.STL
- link link_5: geometry collision mesh filename=./meshes/link_5.STL; visual mesh filename=./meshes/link_5.STL
- link link_6: geometry collision mesh filename=./meshes/link_6.STL; visual mesh filename=./meshes/link_6.STL

Commit message: separate arm parts to links and motor links
Separate robot arm body parts to links and motors for visualization and using the inertial from links and motors combined generated from another URDF file to keep physical properties.

File: simulation/follower.urdf (robot description, URDF)
Before this commit: robot follower, 7 links, 6 joints
Links:
- link base_link: mass 0.024929 -> 0.067266; geometry collision mesh filename=package://follower/meshes/base_link.STL; collision mesh filename=package://follower/meshes/base_link_motor.STL
- link link_1: mass 0.006884 -> 0.05014; geometry collision mesh filename=package://follower/meshes/link_1.STL; collision mesh filename=package://follower/meshes/link_1_motor.STL
- link link_2: mass 0.034312 -> 0.050177; geometry collision mesh filename=package://follower/meshes/link_2.STL; collision mesh filename=package://follower/meshes/link_2_motor.STL
- link link_3: mass 0.047925 -> 0.06379; geometry collision mesh filename=package://follower/meshes/link_3.STL; collision mesh filename=package://follower/meshes/link_3_motor.STL
- link link_4: mass 0.0045392 -> 0.019805; geometry collision mesh filename=package://follower/meshes/link_4.STL; collision mesh filename=package://follower/meshes/link_4_motor.STL
- link link_5: mass 0.013412 -> 0.029277; geometry collision mesh filename=package://follower/meshes/link_5.STL; collision mesh filename=package://follower/meshes/link_5_motor.STL
- link link_6: geometry collision mesh filename=package://follower/meshes/link_6.STL; visual mesh filename=package://follower/meshes/link_6.STL
